Commit message: 5 DOF Arm update.

File: urdf/robot.urdf (robot description, URDF)
Before this commit: robot simple_robot, 6 links, 5 joints
Links:
- added link sixth_link; visual box size=0.05 0.2 0.05
- link fourth_link: geometry visual box size=0.1 0.1 0.1
Joints:
- added joint joint_6: type revolute, parent fourth_link, child sixth_link, origin xyz=-0.05 0.05 0, axis 0 0 1, limit lower=-0.6 upper=0.2 effort=300 velocity=2.0, mimic joint=joint_5 multiplier=-1.0
- joint joint_2: limit lower=-5 upper=5 effort=300 velocity=2.0 -> lower=-0.5 upper=0.5 effort=300 velocity=2.0
- joint joint_3: limit lower=-5 upper=5 effort=300 velocity=2.0 -> lower=-0.5 upper=0.5 effort=300 velocity=2.0
- joint joint_4: axis 0 0 1 -> 0 1 0; limit lower=-0.6 upper=0.18 effort=300 velocity=2.0 -> lower=-0.9 upper=0.9 effort=300 velocity=2.0; origin xyz=0.05 0.5 0 -> xyz=0.0 0.5 0
- joint joint_5: limit lower=-0.6 upper=0.2 effort=300 velocity=2.0 -> lower=-0.6 upper=0.18 effort=300 velocity=2.0; mimic joint=joint_4 multiplier=-1.0 -> (none); origin xyz=-0.05 0.5 0 -> xyz=0.05 0.05 0; parent third_link -> fourth_link
